Commit message: phase 1 fix: resolve mesh paths for IsaacGym, left elbow effort 9->58

File: description/robots/phybot_c2/phybot_c2.urdf (robot description, URDF)
Before this commit: robot phybot_c2, 25 links, 24 joints
Links:
- link base_link: geometry collision sphere radius=0.07; visual mesh filename=meshes/base_link.STL
- link left_ankle_pitch: geometry collision sphere radius=0.045; visual mesh filename=meshes/left_ankle_pitch.STL
- link left_ankle_roll: geometry collision cylinder length=0.24 radius=0.012; collision cylinder length=0.24 radius=0.012
- link left_elbow_pitch: geometry collision cylinder length=0.22 radius=0.035; visual mesh filename=meshes/left_elbow_pitch.STL
- link left_hip_pitch: geometry collision mesh filename=meshes/left_hip_pitch.STL; visual mesh filename=meshes/left_hip_pitch.STL
- link left_hip_roll: geometry collision sphere radius=0.05; visual mesh filename=meshes/left_hip_roll.STL
- link left_hip_yaw: geometry collision cylinder length=0.18 radius=0.04; visual mesh filename=meshes/left_hip_yaw.STL
- link left_knee: geometry collision cylinder length=0.16 radius=0.04; visual mesh filename=meshes/left_knee.STL
- link left_shoulder_pitch: geometry visual mesh filename=meshes/left_shoulder_pitch.STL
- link left_shoulder_roll: geometry collision sphere radius=0.05; visual mesh filename=meshes/left_shoulder_roll.STL
- link left_shoulder_yaw: geometry collision cylinder length=0.14 radius=0.03; visual mesh filename=meshes/left_shoulder_yaw.STL
- link neck_pitch: geometry collision sphere radius=0.07; visual mesh filename=meshes/neck_pitch.STL
- link neck_yaw: geometry visual mesh filename=meshes/neck_yaw.STL
- link right_ankle_pitch: geometry collision sphere radius=0.045; visual mesh filename=meshes/right_ankle_pitch.STL
- link right_ankle_roll: geometry collision cylinder length=0.24 radius=0.012; collision cylinder length=0.24 radius=0.012
- link right_elbow_pitch: geometry collision cylinder length=0.22 radius=0.035; visual mesh filename=meshes/right_elbow_pitch.STL
- link right_hip_pitch: geometry collision mesh filename=meshes/right_hip_pitch.STL; visual mesh filename=meshes/right_hip_pitch.STL
- link right_hip_roll: geometry collision sphere radius=0.05; visual mesh filename=meshes/right_hip_roll.STL
- link right_hip_yaw: geometry collision cylinder length=0.18 radius=0.04; visual mesh filename=meshes/right_hip_yaw.STL
- link right_knee: geometry collision cylinder length=0.16 radius=0.04; visual mesh filename=meshes/right_knee.STL
- link right_shoulder_pitch: geometry visual mesh filename=meshes/right_shoulder_pitch.STL
- link right_shoulder_roll: geometry collision sphere radius=0.05; visual mesh filename=meshes/right_shoulder_roll.STL
- link right_shoulder_yaw: geometry collision cylinder length=0.14 radius=0.03; visual mesh filename=meshes/right_shoulder_yaw.STL
- link torso: geometry collision box size=0.14 0.18 0.28; visual mesh filename=meshes/torso.STL
- link waist_yaw: geometry visual mesh filename=meshes/waist_yaw.STL
Joints:
- joint left_elbow_pitch: limit lower=-2.36 upper=0 effort=9 velocity=98.16 -> lower=-2.36 upper=0 effort=58 velocity=98.16

Commit message: phase 5: kongti training tweaks, motionframe ref obs, traced jit export
- domain_rand: base mass randomization now targets an explicit base_mass_link
  (phybot has neither pelvis nor torso_link; waist_yaw is the real trunk after
  collapse_fixed_joints), with an assert against negative mass in isaacgym.py
- obs: add local_ref_rigid_body_pos_motionframe, a pure feed-forward reference
  anchored on env origin rather than the robot root
- rewards: add teleop_jump_height, paid only while the reference is airborne;
  loosen torque/dof-pos soft limits and action-rate penalty for kongti
- fix terminate_when_dof_far reducing over the wrong dim (any over a scalar norm)
- eval_agent: also export a TorchScript-traced _deploy.pt for the C++ libtorch
  deployment in PhybotSoftware RL_deploy_*
- urdf: shorten ankle collision cylinders, fix neck_pitch inertial origin z

File: description/robots/phybot_c2/phybot_c2.urdf (robot description, URDF)
Before this commit: robot phybot_c2, 25 links, 24 joints
Links:
- link left_ankle_roll: geometry collision cylinder length=0.18 radius=0.012; collision cylinder length=0.18 radius=0.012
- link right_ankle_roll: geometry collision cylinder length=0.18 radius=0.012; collision cylinder length=0.18 radius=0.012
