Commit message: phase 6: mujoco sim2sim deployment, phybot asset variants, motion tooling
- deploy: URCI/MuJoCo sim2sim path (base_urci.yaml, urci.py, deploy/mujoco.py,
  deploy/urcirobot.py) for running trained policies outside IsaacGym
- export_ref_motionframe.py: dump the 75-dim local_ref_rigid_body_pos_motionframe
  table (row k = motion((k+1)*dt)) for the C++ deployment side
- phybot_c2 assets: add phybot_c2.xml (MuJoCo), phybot_c2_hll.urdf and
  phybot_c2_32kg.urdf variants; fk consistency check updated
- domain rand: base_com_link fallback docs, phybot DR configs (main_phybot,
  dr_nil_phybot), unit comment fix on base_com_range (m, not kg)
- motion tooling: gmr_npz_to_pkl_g1.py converter, edit_motion.py
- analysis_plot_eval_joints callback for per-joint eval plots
- gitignore URCI eval output dirs (example/*/motions/)

Co-Authored-By: Claude Opus 5 <noreply@anthropic.com>

File: description/robots/phybot_c2/phybot_c2_32kg.urdf (robot description, URDF)
Before this commit: robot phybot_c2, 27 links, 26 joints
Links:
- removed link left_wrist_yaw
- removed link right_wrist_yaw
- link base_link: mass 7.2436 -> 3.2436
- link left_ankle_roll: geometry collision cylinder length=0.18 radius=0.012; collision cylinder length=0.18 radius=0.012
- link left_hip_pitch: geometry collision mesh filename=meshes/left_hip_pitch.STL; visual mesh filename=meshes/left_hip_pitch.STL
- link neck_pitch: mass 0.05 -> 2.36
- link right_ankle_roll: geometry collision cylinder length=0.18 radius=0.012; collision cylinder length=0.18 radius=0.012
- link right_hip_pitch: geometry collision mesh filename=meshes/right_hip_pitch.STL; visual mesh filename=meshes/right_hip_pitch.STL
- link torso: mass 11.89499645954187 -> 7.89499645954187
Joints:
- removed joint left_wrist_yaw
- removed joint right_wrist_yaw
- joint left_ankle_pitch: limit lower=-1.57 upper=1.57 effort=90 velocity=98.37 -> lower=-1.57 upper=1.57 effort=58 velocity=98.37
- joint left_ankle_roll: limit lower=-1.13 upper=1.13 effort=90 velocity=98.37 -> lower=-1.13 upper=1.13 effort=58 velocity=98.37
- joint left_elbow_pitch: limit lower=-2.36 upper=0 effort=90 velocity=98.16 -> lower=-2.36 upper=0 effort=58 velocity=98.16
- joint left_hip_pitch: limit lower=-3.05 upper=2.09 effort=160 velocity=99.21 -> lower=-3.05 upper=2.09 effort=200 velocity=99.21
- joint left_hip_roll: limit lower=-0.44 upper=3.05 effort=100 velocity=98.9 -> lower=-0.44 upper=3.05 effort=80 velocity=98.9
- joint left_hip_yaw: limit lower=-2.53 upper=2.53 effort=90 velocity=98.37 -> lower=-2.53 upper=2.53 effort=58 velocity=98.37
- joint left_knee: limit lower=-0.05 upper=2.36 effort=100 velocity=98.9 -> lower=-0.05 upper=2.36 effort=80 velocity=98.9
- joint left_shoulder_pitch: limit lower=-3.14 upper=3.14 effort=90 velocity=98.37 -> lower=-3.58 upper=2.01 effort=58 velocity=98.37
- joint left_shoulder_roll: limit lower=-3.14 upper=3.14 effort=90 velocity=98.37 -> lower=-0.35 upper=3.05 effort=58 velocity=98.37
- joint left_shoulder_yaw: limit lower=-3.14 upper=3.14 effort=90 velocity=98.37 -> lower=-2.53 upper=2.53 effort=58 velocity=98.37
- joint neck_pitch: limit lower=-0.61 upper=0.61 effort=30 velocity=98.16 -> lower=-0.61 upper=0.61 effort=9 velocity=98.16
- joint neck_yaw: limit lower=-2.62 upper=2.62 effort=30 velocity=98.16 -> lower=-2.62 upper=2.62 effort=9 velocity=98.16
- joint right_ankle_pitch: limit lower=-1.57 upper=1.57 effort=90 velocity=98.37 -> lower=-1.57 upper=1.57 effort=58 velocity=98.37
- joint right_ankle_roll: limit lower=-1.13 upper=1.13 effort=90 velocity=98.37 -> lower=-1.13 upper=1.13 effort=58 velocity=98.37
- joint right_elbow_pitch: limit lower=-2.36 upper=0 effort=90 velocity=98.37 -> lower=-2.36 upper=0 effort=58 velocity=98.37
- joint right_hip_pitch: limit lower=-3.05 upper=2.09 effort=160 velocity=99.21 -> lower=-3.05 upper=2.09 effort=200 velocity=99.21
- joint right_hip_roll: limit lower=-3.05 upper=0.44 effort=100 velocity=98.9 -> lower=-3.05 upper=0.44 effort=80 velocity=98.9
- joint right_hip_yaw: limit lower=-2.53 upper=2.53 effort=90 velocity=98.37 -> lower=-2.53 upper=2.53 effort=58 velocity=98.37
- joint right_knee: limit lower=-0.05 upper=2.36 effort=100 velocity=98.9 -> lower=-0.05 upper=2.36 effort=80 velocity=98.9
- joint right_shoulder_pitch: limit lower=-3.14 upper=3.14 effort=90 velocity=98.37 -> lower=-3.58 upper=2.01 effort=58 velocity=98.37
- joint right_shoulder_roll: limit lower=-3.14 upper=3.14 effort=90 velocity=98.37 -> lower=-3.05 upper=0.35 effort=58 velocity=98.37
- joint right_shoulder_yaw: limit lower=-3.14 upper=3.14 effort=90 velocity=98.37 -> lower=-2.53 upper=2.53 effort=58 velocity=98.37
- joint waist_yaw: limit lower=-2.62 upper=2.62 effort=90 velocity=98.37 -> lower=-2.62 upper=2.62 effort=58 velocity=98.37

File: description/robots/phybot_c2/phybot_c2_hll.urdf (robot description, URDF)
Before this commit: robot phybot_c2, 27 links, 26 joints
Links:
- removed link left_wrist_yaw
- removed link right_wrist_yaw
- link base_link: mass 7.2436 -> 3.2436
- link left_ankle_roll: geometry collision cylinder length=0.18 radius=0.012; collision cylinder length=0.18 radius=0.012
- link left_hip_pitch: geometry collision mesh filename=meshes/left_hip_pitch.STL; visual mesh filename=meshes/left_hip_pitch.STL
- link neck_pitch: mass 0.05 -> 1.4368
- link right_ankle_roll: geometry collision cylinder length=0.18 radius=0.012; collision cylinder length=0.18 radius=0.012
- link right_hip_pitch: geometry collision mesh filename=meshes/right_hip_pitch.STL; visual mesh filename=meshes/right_hip_pitch.STL
- link torso: mass 11.89499645954187 -> 7.89499645954187
Joints:
- removed joint left_wrist_yaw
- removed joint right_wrist_yaw
- joint left_ankle_pitch: limit lower=-1.57 upper=1.57 effort=90 velocity=98.37 -> lower=-1.57 upper=1.57 effort=58 velocity=98.37
- joint left_ankle_roll: limit lower=-1.13 upper=1.13 effort=90 velocity=98.37 -> lower=-1.13 upper=1.13 effort=58 velocity=98.37
- joint left_elbow_pitch: limit lower=-2.36 upper=0 effort=90 velocity=98.16 -> lower=-2.36 upper=0 effort=58 velocity=98.16
- joint left_hip_pitch: limit lower=-3.05 upper=2.09 effort=160 velocity=99.21 -> lower=-3.05 upper=2.09 effort=200 velocity=99.21
- joint left_hip_roll: limit lower=-0.44 upper=3.05 effort=100 velocity=98.9 -> lower=-0.44 upper=3.05 effort=80 velocity=98.9
- joint left_hip_yaw: limit lower=-2.53 upper=2.53 effort=90 velocity=98.37 -> lower=-2.53 upper=2.53 effort=58 velocity=98.37
- joint left_knee: limit lower=-0.05 upper=2.36 effort=100 velocity=98.9 -> lower=-0.05 upper=2.36 effort=80 velocity=98.9
- joint left_shoulder_pitch: limit lower=-3.14 upper=3.14 effort=90 velocity=98.37 -> lower=-3.58 upper=2.01 effort=58 velocity=98.37
- joint left_shoulder_roll: limit lower=-3.14 upper=3.14 effort=90 velocity=98.37 -> lower=-0.35 upper=3.05 effort=58 velocity=98.37
- joint left_shoulder_yaw: limit lower=-3.14 upper=3.14 effort=90 velocity=98.37 -> lower=-2.53 upper=2.53 effort=58 velocity=98.37
- joint neck_pitch: limit lower=-0.61 upper=0.61 effort=30 velocity=98.16 -> lower=-0.61 upper=0.61 effort=9 velocity=98.16
- joint neck_yaw: limit lower=-2.62 upper=2.62 effort=30 velocity=98.16 -> lower=-2.62 upper=2.62 effort=9 velocity=98.16
- joint right_ankle_pitch: limit lower=-1.57 upper=1.57 effort=90 velocity=98.37 -> lower=-1.57 upper=1.57 effort=58 velocity=98.37
- joint right_ankle_roll: limit lower=-1.13 upper=1.13 effort=90 velocity=98.37 -> lower=-1.13 upper=1.13 effort=58 velocity=98.37
- joint right_elbow_pitch: limit lower=-2.36 upper=0 effort=90 velocity=98.37 -> lower=-2.36 upper=0 effort=58 velocity=98.37
- joint right_hip_pitch: limit lower=-3.05 upper=2.09 effort=160 velocity=99.21 -> lower=-3.05 upper=2.09 effort=200 velocity=99.21
- joint right_hip_roll: limit lower=-3.05 upper=0.44 effort=100 velocity=98.9 -> lower=-3.05 upper=0.44 effort=80 velocity=98.9
- joint right_hip_yaw: limit lower=-2.53 upper=2.53 effort=90 velocity=98.37 -> lower=-2.53 upper=2.53 effort=58 velocity=98.37
- joint right_knee: limit lower=-0.05 upper=2.36 effort=100 velocity=98.9 -> lower=-0.05 upper=2.36 effort=80 velocity=98.9
- joint right_shoulder_pitch: limit lower=-3.14 upper=3.14 effort=90 velocity=98.37 -> lower=-3.58 upper=2.01 effort=58 velocity=98.37
- joint right_shoulder_roll: limit lower=-3.14 upper=3.14 effort=90 velocity=98.37 -> lower=-3.05 upper=0.35 effort=58 velocity=98.37
- joint right_shoulder_yaw: limit lower=-3.14 upper=3.14 effort=90 velocity=98.37 -> lower=-2.53 upper=2.53 effort=58 velocity=98.37
- joint waist_yaw: limit lower=-2.62 upper=2.62 effort=90 velocity=98.37 -> lower=-2.62 upper=2.62 effort=58 velocity=98.37
