Commit message: phybot_c2: G1 actuator params (effort/vel limit, armature), PD experiments

File: description/robots/phybot_c2/phybot_c2_hll.urdf (robot description, URDF)
Before this commit: robot phybot_c2, 25 links, 24 joints
Links:
- link left_ankle_roll: geometry collision cylinder length=0.24 radius=0.012; collision cylinder length=0.24 radius=0.012
- link right_ankle_roll: geometry collision cylinder length=0.24 radius=0.012; collision cylinder length=0.24 radius=0.012
